Commit message: adapted the path to some resources
but it still needs editing when run on another system

File: meshes/cinempc.urdf (robot description, URDF)
Before this commit: robot iris, 1 links, 0 joints
Links:
- link base_link: geometry visual mesh filename=file:///home/cconradi/Documents/catkin_ws/src/nav_stack/mes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 scale=0.001 0.001 0.001
